File: src/MainBoard.kicad_sch (KiCad schematic)
At the start: 64 parts, among them J3 ISP Port, J48 1-726388-2, J49 1-726388-2, J5 MiniFit_2x10_F, J50 1-726388-2, J51 1-726388-2, J52 1-726388-2, J53 1-726388-2, J54 1-726388-2, J55 1-726388-2, K1 RAYEX-L90S, K2 RAYEX-L90S, K3 RAYEX-L90S, Q1 2N7002, Q2 2N7002, Q3 2N7002, Q4 2N7002, U1 ATtiny84-20P, U2 LM2576HVT-ADJ

Commit message: Update Schematics design
Parts:
- removed C1: 100nF, Capacitor_THT:C_Disc_D5.0mm_W2.5mm_P5.00mm, symbol Device:C
- removed D1: BZX79C2V7, Diode_SMD:D_MiniMELF, symbol Diode:BZV55C2V7
- removed D4, D5: SK510, Diode_SMD:D_SMB_Handsoldering, symbol Diode:1N5400
- removed D6, D8: BZX79C2V7, Diode_SMD:D_MiniMELF, symbol Diode:BZV55C3V0
- removed F?: 12V 30A, symbol Device:Fuse
- removed F?: 12V 20A, symbol Device:Fuse
- removed F?: 12V 10A, symbol Device:Fuse
- removed F? (x2): 12V 15A, symbol Device:Fuse
- removed F?: 12V 3A, symbol Device:Fuse
- removed J3: ISP Port, Connector_PinSocket_2.54mm:PinSocket_2x03_P2.54mm_Vertical_SMD, symbol Connector_Generic:Conn_02x03_Odd_Even
- removed J48, J49, J50, J51, J52, J53, J54, J55: 1-726388-2, 17263882, symbol SamacSys_Parts:1-726388-2
- removed J5: MiniFit_2x10_F, Connector_Molex:Molex_Mini-Fit_Jr_5566-20A_2x10_P4.20mm_Vertical, symbol Connector_Generic:Conn_02x10_Counter_Clockwise
- removed JP1, JP2, JP3: Jumper_2_Bridged, symbol Jumper:Jumper_2_Bridged
- removed Q1, Q2, Q3: 2N7002, Package_TO_SOT_SMD:SOT-23, symbol Transistor_FET:2N7002
- removed R? (x2): 1.5K, Resistor_SMD:R_1206_3216Metric_Pad1.30x1.75mm_HandSolder, symbol Device:R
- removed R? (x4): 15K, Resistor_SMD:R_1206_3216Metric_Pad1.30x1.75mm_HandSolder, symbol Device:R
- removed R? (x9): 10K, Resistor_SMD:R_1206_3216Metric_Pad1.30x1.75mm_HandSolder, symbol Device:R
- removed U1: ATtiny84-20P, Package_DIP:DIP-14_W7.62mm, symbol MCU_Microchip_ATtiny:ATtiny84-20P
- added C?: 100nF, Capacitor_THT:C_Disc_D5.0mm_W2.5mm_P5.00mm, symbol Device:C
- added D2, D4, D5: BZX79C2V7, Diode_SMD:D_MiniMELF, symbol Diode:BZV55C2V7
- added F?: 12V 3A, symbol Device:Fuse
- added F?: 12V 30A, symbol Device:Fuse
- added F?: 12V 20A, symbol Device:Fuse
- added F?: 12V 15A, symbol Device:Fuse
- added F?: 12V 10A, symbol Device:Fuse
- added J1, J10, J11, J12, J2, J3, J4, J5, J8, J9: 1217080-1, 1217080-1, symbol SamacSys_Parts:1217080-1
- added J13: MiniFit_2x09_F, Connector_Molex:Molex_Mini-Fit_Jr_5566-18A_2x09_P4.20mm_Vertical, symbol Connector_Generic:Conn_02x09_Counter_Clockwise
- added Q1, Q7: BC547, Package_TO_SOT_THT:TO-92_Inline, symbol Transistor_BJT:BC547
- added Q10: BC557, Package_TO_SOT_THT:TO-92_Inline, symbol Transistor_BJT:BC557
- added Q11, Q3: IRF530, TO255P460X1020X2008-3P, symbol SamacSys_Parts:IRF530
- added Q5, Q6, Q8: 2N7002, Package_TO_SOT_SMD:SOT-23, symbol Transistor_FET:2N7002
- added Q?: BPW96B, LED_THT:LED_D5.0mm, symbol Device:Q_Photo_NPN
- added R? (x7): 10K, Resistor_SMD:R_1206_3216Metric_Pad1.30x1.75mm_HandSolder, symbol Device:R
- added R? (x2): 33K, Resistor_SMD:R_1206_3216Metric_Pad1.30x1.75mm_HandSolder, symbol Device:R
- added R?: 1K, Resistor_THT:R_Axial_DIN0204_L3.6mm_D1.6mm_P5.08mm_Horizontal, symbol Device:R
- added U1: ATtiny85-20P, Package_DIP:DIP-8_W7.62mm, symbol MCU_Microchip_ATtiny:ATtiny85-20P
- RV1: value 10K -> 100K
- RV2: value 10K -> 47K
- renumbered D2 to D1, D7 to D6, D9 to D7
Connections:
- net +12V: now also F?.2, F?.2, J3.1, J3.2, J4.1, J4.2, Q10.1 (C), R?.1, R?.1
- net +5V: now also C?.1, J13.5 (Pin_5), Q1.1 (C), R?.1, U1.8 (VCC); no longer RV2.1
- net +BATT: now also F?.1, F?.1, F?.1, J13.1 (Pin_1), J2.1, J2.2, J5.1, J5.2, J8.1, J8.2
- net +VDC: now also F?.2, J1.1, J1.2
- net ABeam1: now also J13.13 (Pin_13)
- net ABeam2: now also J13.11 (Pin_11)
- net AuxSwitch1: now also J13.12 (Pin_12)
- net AuxSwitch2: now also J13.10 (Pin_10)
- net EBlinker: now also J13.6 (Pin_6), R?.1
- net GND: now also D2.2 (A), D5.2 (A), Q11.3, Q3.3, Q6.2 (S); no longer C?.2, C?.2, D3.2 (A), D?.2 (A), Q4.2 (S), R?.2, RV2.3, U2.3 (GND), U2.5 (~{ON}/OFF)
- net Key: now also J13.7 (Pin_7), R?.1
- net Killswitch: now also J13.8 (Pin_8), R?.2
- net LowBat: now also J13.9 (Pin_9), Q10.3 (E)
- net PLight: now also J13.14 (Pin_14)
- net VInst: now also F?.2, J12.1, J12.2, J13.4 (Pin_4)
- net VLight: now also F?.1, J11.1, J11.2, J13.2 (Pin_2)
- net VOutlet: now also F?.1, J10.1, J10.2
- net VRadio: now also F?.2, J13.3 (Pin_3), J9.1, J9.2
- net at Q4.1 (G): now also D3.1 (K), R?.2
- net GNDRelay: now reaches D1.2 (A), K1.A2
- net GNDRelay: now also Q5.3 (D)
- net GND2 renamed GNDDash
- net GNDDash: now also J13.18 (Pin_18)
- net LightIntensityPot: no longer names the net of RV1.2
- net LightIntensityPot: now also U1.7 (PB2)
- net LightSensorPot: no longer names the net of RV2.2
- net LightSensorPot: now also Q7.2 (B)
- new net: D5.1 (K), Q11.1, Q6.1 (G), R?.2
- new net: Q5.2 (S), Q6.3 (D)
- new net: Q1.2 (B), Q?.1 (C), R?.2
- new net: Q10.2 (B), Q7.1 (C), R?.2
- new net: R?.1, R?.2, R?.2, U1.3 (XTAL2/PB4)
- new net: D4.1 (K), Q8.1 (G), R?.2
- new net: R?.2, RV2.3
- new net: Q1.3 (E), U1.2 (XTAL1/PB3)
- new net: D2.1 (K), Q3.1, Q5.1 (G), R?.1
- new net DimmerDash: R?.1, U1.5 (AREF/PB0)
- new net DimmerEBlinker: R?.1, U1.6 (PB1)
- new net GND5: C?.2, C?.2, C?.2, D3.2 (A), D4.2 (A), D?.2 (A), Q11.2, Q4.2 (S), Q7.3 (E), Q8.2 (S), Q?.2 (E), R?.1, R?.2, R?.2, RV2.1, U1.4 (GND), U2.3 (GND), U2.5 (~{ON}/OFF)
- new net GNDEBlinker: J13.17 (Pin_17), Q8.3 (D)
- new net GNDRadio: J13.16 (Pin_16), Q3.2
- no-connect marks 6 -> 2
Other:
- note added: "Kill Switch control"
- note added: "Lights Dimmer"
- note added: "Low Battery indicator"
- note removed: "Adjustment Pots"
- note removed: "Battery Sensor"
- note removed: "Dimmer control"
- note removed: "Emergency Stop"
- note removed: "ISP Port"
- note removed: "Light sensor sensitivity"
- note removed: "Lights Sensors"
- note removed: "Lights intensity"
- moved on the sheet: C?, D1, D?, J?, K1, L?, R?, U2

Commit message: Update schematic design
Connections:
- net AuxSwitch1: now also D6.1 (K); no longer D6.2 (A)
- net AuxSwitch2: now also D7.1 (K); no longer D7.2 (A)
- net GND: now also D6.2 (A), D7.2 (A); no longer D6.1 (K), D7.1 (K)
Changed lines of the file:
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@@
+    )
+  )
+  (symbol (lib_id "Diode:US1M") (at 201.93 52.07 180) (unit 1)
+    (in_bom yes) (on_board yes) (dnp no) (fields_autoplaced)
+    (property "Reference" "D6" (at 201.93 46.99 0)
+      (effects (font (size 1.27 1.27)))
+    )
+    (property "Value" "US1M" (at 201.93 49.53 0)
+      (effects (font (size 1.27 1.27)))
+    )
+    (property "Footprint" "Diode_SMD:D_SMA" (at 201.93 47.625 0)
+      (effects (font (size 1.27 1.27)) hide)
+    )
+    (property "Datasheet" "https://www.diodes.com/assets/Datasheets/ds16008.pdf" (at 201.93 52.07 0)
+      (effects (font (size 1.27 1.27)) hide)
+    )
+    (property "Sim.Device" "D" (at 201.93 52.07 0)
+      (effects (font (size 1.27 1.27)) hide)
+    )
+    (property "Sim.Pins" "1=K 2=A" (at 201.93 52.07 0)
+      (effects (font (size 1.27 1.27)) hide)
+    )
+    (property "Vendor" "Mauser" (at 201.93 52.07 0)
+      (effects (font (size 1.27 1.27)) hide)
+    )
+    (property "Vendor Link" "https://mauser.pt/catalog/product_info.php?products_id=007-0391" (at 201.93 52.07 0)
+      (effects (font (size 1.27 1.27)) hide)
+    )
+    (property "Vendor Ref" "007-0391" (at 201.93 52.07 0)
+      (effects (font (size 1.27 1.27)) hide)
+    )
+    (pin "1")
+    (pin "2")
+    (instances
+      (project "dragstar-infotainment"
+        (path "/e63e39d7-6ac0-4ffd-8aa3-1841a4541b55/5d40715c-dfc9-4b95-9cc7-adbd4b609d9b"
+          (reference "D6") (unit 1)
+        )
+      )
     )
   )
@@
     )
   )
-  (symbol (lib_id "Diode:US1M") (at 201.93 52.07 0) (unit 1)
-    (in_bom yes) (on_board yes) (dnp no) (fields_autoplaced)
-    (property "Reference" "D6" (at 201.93 46.99 0)
-      (effects (font (size 1.27 1.27)))
-    )
-    (property "Value" "US1M" (at 201.93 49.53 0)
-      (effects (font (size 1.27 1.27)))
-    )
-    (property "Footprint" "Diode_SMD:D_SMA" (at 201.93 56.515 0)
-      (effects (font (size 1.27 1.27)) hide)
-    )
-    (property "Datasheet" "https://www.diodes.com/assets/Datasheets/ds16008.pdf" (at 201.93 52.07 0)
-      (effects (font (size 1.27 1.27)) hide)
-    )
-    (property "Sim.Device" "D" (at 201.93 52.07 0)
-      (effects (font (size 1.27 1.27)) hide)
-    )
-    (property "Sim.Pins" "1=K 2=A" (at 201.93 52.07 0)
-      (effects (font (size 1.27 1.27)) hide)
-    )
-    (property "Vendor" "Mauser" (at 201.93 52.07 0)
-      (effects (font (size 1.27 1.27)) hide)
-    )
-    (property "Vendor Link" "https://mauser.pt/catalog/product_info.php?products_id=007-0391" (at 201.93 52.07 0)
-      (effects (font (size 1.27 1.27)) hide)
-    )
-    (property "Vendor Ref" "007-0391" (at 201.93 52.07 0)
-      (effects (font (size 1.27 1.27)) hide)
-    )
-    (pin "1")
-    (pin "2")
-    (instances
-      (project "dragstar-infotainment"
-        (path "/e63e39d7-6ac0-4ffd-8aa3-1841a4541b55/5d40715c-dfc9-4b95-9cc7-adbd4b609d9b"
-          (reference "D6") (unit 1)
-        )
-      )
-    )
-  )
   (symbol (lib_id "Diode:BZV55C2V7") (at 110.49 175.26 90) (mirror x) (unit 1)
     (in_bom yes) (on_board yes) (dnp no)
@@
     )
   )
-  (symbol (lib_id "Diode:US1M") (at 252.73 52.07 0) (unit 1)
+  (symbol (lib_id "Diode:US1M") (at 252.73 52.07 180) (unit 1)
     (in_bom yes) (on_board yes) (dnp no) (fields_autoplaced)
     (property "Reference" "D7" (at 252.73 46.99 0)
@@
       (effects (font (size 1.27 1.27)))
     )
-    (property "Footprint" "Diode_SMD:D_SMA" (at 252.73 56.515 0)
-      (effects (font (size 1.27 1.27)) hide)
-    )
+    (property "Footprint" "Diode_SMD:D_SMA" (at 252.73 47.625 0)
+      (effects (font (size 1.27 1.27)) hide)
+    )
