File: src/dragstar-infotainment.kicad_pcb (KiCad board)
At the start: 2 copper layers, 51 parts, among them J1 XT60-M, J3 ISP Port, J4 Barrel_Jack, J48 1-726388-2, J49 1-726388-2, J50 1-726388-2, J51 1-726388-2, J52 1-726388-2, J53 1-726388-2, J54 1-726388-2, J55 1-726388-2, K1 RAYEX-L90S, K2 RAYEX-L90S, K3 RAYEX-L90S, Q1 2N7002, Q2 2N7002, Q3 2N7002, Q4 2N7002, U1 ATtiny84-20P, U2 LM2576HVT-ADJ

Commit message: Update Schematics design
Parts:
- J3: footprint Connector_PinSocket_2.54mm:PinSocket_2x03_P2.54mm_Vertical_SMD -> Connector_PinSocket_2.54mm:PinSocket_2x03_P2.54mm_Vertical
- renumbered J49 to J10, J48 to J11, J55 to J12, J53 to J13, J54 to J6, J52 to J7, J51 to J8, J50 to J9
Connections:
- J4 pad MP: GND -> (no net)
- U1 pad 3: LightSensorPot -> LightSensor
- U1 pad 5: LightSensor -> unconnected-(U1-PB2-Pad5)

Commit message: update Schematics
Parts:
- removed C1: 100nF, Capacitor_THT:C_Disc_D5.0mm_W2.5mm_P5.00mm
- removed C2: 1nF, Capacitor_THT:C_Disc_D5.0mm_W2.5mm_P5.00mm
- removed C3: 0.1nF, Capacitor_SMD:C_1206_3216Metric_Pad1.33x1.80mm_HandSolder
- removed the J10 at (132.5, 89.7)
- removed the J11 at (152.5, 89.7)
- removed the J13 at (136.8, 117.0)
- removed J3: ISP Port, Connector_PinSocket_2.54mm:PinSocket_2x03_P2.54mm_Vertical
- removed the J6 at (332.2, 140.7)
- removed the J7 at (122.5, 89.7)
- removed the J8 at (162.5, 89.8)
- removed L1: 100µH, Inductor_THT:L_Radial_D9.5mm_P5.00mm_Fastron_07HVP
- removed U2: LM2576HVT-ADJ, Package_TO_SOT_THT:TO-220-5_Vertical
- added BT1: 9V, Connector_JST:JST_XH_B2B-XH-A_1x02_P2.50mm_Vertical, F.Cu at (459.3, 15.0)
- added D11: US1M, Diode_SMD:D_SMA, F.Cu at (432.3, 21.6)
- added D12: BZX79C2V7, Diode_SMD:D_MiniMELF, F.Cu at (405.0, 38.0)
- added D13: LED, LED_THT:LED_D5.0mm, F.Cu at (415.5, 52.6)
- added D14: LED, LED_THT:LED_D5.0mm, F.Cu at (423.0, 52.6)
- added D15: LED, LED_THT:LED_D5.0mm, F.Cu at (430.5, 52.6)
- added D16: LED, LED_THT:LED_D5.0mm, F.Cu at (438.0, 52.6)
- added D17: LED Green, LED_THT:LED_D5.0mm, F.Cu at (462.5, 85.0)
- added D18: LED Blue, LED_THT:LED_D5.0mm, F.Cu at (470.0, 85.0)
- added D19: LED Red, LED_THT:LED_D5.0mm, F.Cu at (455.0, 85.0)
- added D20: LED Yellow, LED_THT:LED_D5.0mm, F.Cu at (477.5, 85.0)
- added D21: LED Green, LED_THT:LED_D5.0mm, F.Cu at (447.5, 85.0)
- added D26: BZX79C2V7, Diode_SMD:D_MiniMELF, F.Cu at (465.5, 21.1)
- added D27: P600A, Diode_THT:D_P600_R-6_P12.70mm_Horizontal, F.Cu at (364.2, 83.3)
- added D28: US1M, Diode_SMD:D_SMA, F.Cu at (112.5, 138.8)
- added D30: BZX79C2V7, Diode_SMD:D_MiniMELF, F.Cu at (120.8, 143.5)
- added J**: 1217080-1, SamacSys_Parts:1217080-1, F.Cu at (107.5, 90.0)
- added J**: 1217080-1, SamacSys_Parts:1217080-1, F.Cu at (185.2, 90.0)
- added J**: 1217080-1, SamacSys_Parts:1217080-1, F.Cu at (112.5, 101.7)
- added J**: 1217080-1, SamacSys_Parts:1217080-1, F.Cu at (192.5, 101.7)
- added J**: 1217080-1, SamacSys_Parts:1217080-1, F.Cu at (192.5, 90.0)
- added J**: 1217080-1, SamacSys_Parts:1217080-1, F.Cu at (185.2, 101.7)
- added J**: 1217080-1, SamacSys_Parts:1217080-1, F.Cu at (112.5, 90.0)
- added J10: MiniFit_2x04_M, Connector_Molex:Molex_Mini-Fit_Jr_5566-08A_2x04_P4.20mm_Vertical, F.Cu at (448.7, 52.1)
- added J10: 1217080-1, SamacSys_Parts:1217080-1, F.Cu at (142.5, 90.0)
- added J11: USB_A, Connector_USB:USB_A_Molex_67643_Horizontal, F.Cu at (470.6, 52.2)
- added J11: 1217080-1, SamacSys_Parts:1217080-1, F.Cu at (172.5, 90.0)
- added J13: 1217080-1, SamacSys_Parts:1217080-1, F.Cu at (132.5, 101.8)
- added J13: MiniFit_2x04_F, Connector_Molex:Molex_Mini-Fit_Jr_5566-08A_2x04_P4.20mm_Vertical, F.Cu at (448.7, 65.2)
- added J14: MiniFit_2x01_M, Connector_Molex:Molex_Mini-Fit_Jr_5566-02A_2x01_P4.20mm_Vertical, F.Cu at (448.7, 105.1)
- added J14: 1217080-1, SamacSys_Parts:1217080-1, F.Cu at (162.5, 101.8)
- added J15: 1217080-1, SamacSys_Parts:1217080-1, F.Cu at (152.5, 101.7)
- added J15: MiniFit_2x01_M, Connector_Molex:Molex_Mini-Fit_Jr_5566-02A_2x01_P4.20mm_Vertical, F.Cu at (456.2, 105.1)
- added J16: MiniFit_2x03_F, Connector_Molex:Molex_Mini-Fit_Jr_5566-06A_2x03_P4.20mm_Vertical, F.Cu at (448.7, 92.0)
- added J16: 1217080-1, SamacSys_Parts:1217080-1, F.Cu at (142.5, 101.6)
- added J17: 1217080-1, SamacSys_Parts:1217080-1, F.Cu at (172.5, 101.8)
- added J2: XT60-M, Connector_AMASS:AMASS_XT60PW-M_1x02_P7.20mm_Horizontal, F.Cu at (106.4, 106.3)
- added J42: MiniFit_2x04_M, Connector_Molex:Molex_Mini-Fit_Jr_5566-08A_2x04_P4.20mm_Vertical, F.Cu at (459.5, -0.13)
- added J44: MiniFit_2x02_M, Connector_Molex:Molex_Mini-Fit_Jr_5566-04A_2x02_P4.20mm_Vertical, F.Cu at (372.8, 41.0)
- added J45: MiniFit_2x03_M, Connector_Molex:Molex_Mini-Fit_Jr_5566-06A_2x03_P4.20mm_Vertical, F.Cu at (356.9, -0.13)
- added J46: MiniFit_2x03_M, Connector_Molex:Molex_Mini-Fit_Jr_5566-06A_2x03_P4.20mm_Vertical, F.Cu at (356.9, 12.9)
- added J47: MiniFit_2x03_M, Connector_Molex:Molex_Mini-Fit_Jr_5566-06A_2x03_P4.20mm_Vertical, F.Cu at (356.9, 26.0)
- added J48: MiniFit_2x04_M, Connector_Molex:Molex_Mini-Fit_Jr_5566-08A_2x04_P4.20mm_Vertical, F.Cu at (372.8, 14.9)
- added J49: MiniFit_2x03_M, Connector_Molex:Molex_Mini-Fit_Jr_5566-06A_2x03_P4.20mm_Vertical, F.Cu at (356.9, 39.0)
- added J5: MiniFit_2x03_F, Connector_Molex:Molex_Mini-Fit_Jr_5566-06A_2x03_P4.20mm_Vertical, F.Cu at (400.9, 65.2)
- added J50: MiniFit_2x03_M, Connector_Molex:Molex_Mini-Fit_Jr_5566-06A_2x03_P4.20mm_Vertical, F.Cu at (356.9, 52.1)
- added J51: MiniFit_2x01_F, Connector_Molex:Molex_Mini-Fit_Jr_5566-02A_2x01_P4.20mm_Vertical, F.Cu at (372.8, 28.0)
- added J53: Barrel_Jack, Connector_BarrelJack:BarrelJack_CUI_PJ-063AH_Horizontal, F.Cu at (375.6, -1.38)
- added J54: Barrel_Jack, Connector_BarrelJack:BarrelJack_CUI_PJ-063AH_Horizontal, F.Cu at (388.6, -1.38)
- added J55: MiniFit_2x01_F, Connector_Molex:Molex_Mini-Fit_Jr_5566-02A_2x01_P4.20mm_Vertical, F.Cu at (380.2, 28.0)
- added J57: 1217080-1, SamacSys_Parts:1217080-1, F.Cu at (357.5, 65.4)
- added J58: 1217080-1, SamacSys_Parts:1217080-1, F.Cu at (357.5, 68.6)
- added J59: 1217080-1, SamacSys_Parts:1217080-1, F.Cu at (357.5, 71.8)
- added J6: MiniFit_2x03_F, Connector_Molex:Molex_Mini-Fit_Jr_5566-06A_2x03_P4.20mm_Vertical, F.Cu at (400.9, 78.2)
- added J6: 1217080-1, SamacSys_Parts:1217080-1, F.Cu at (122.5, 101.7)
- added J60: 1217080-1, SamacSys_Parts:1217080-1, F.Cu at (357.5, 75.0)
- added J61: 1217080-1, SamacSys_Parts:1217080-1, F.Cu at (357.5, 78.2)
- added J62: 1217080-1, SamacSys_Parts:1217080-1, F.Cu at (357.5, 81.4)
- added J63: 1217080-1, SamacSys_Parts:1217080-1, F.Cu at (357.5, 84.6)
- added J64: 1217080-1, SamacSys_Parts:1217080-1, F.Cu at (357.5, 87.8)
- added J65: 1217080-1, SamacSys_Parts:1217080-1, F.Cu at (357.5, 91.0)
- added J66: 1217080-1, SamacSys_Parts:1217080-1, F.Cu at (357.5, 94.2)
- added J67: 1217080-1, SamacSys_Parts:1217080-1, F.Cu at (357.5, 97.4)
- added J68: 1217080-1, SamacSys_Parts:1217080-1, F.Cu at (357.5, 100.6)
- added J7: 1217080-1, SamacSys_Parts:1217080-1, F.Cu at (132.5, 90.0)
- added J7: MiniFit_2x03_F, Connector_Molex:Molex_Mini-Fit_Jr_5566-06A_2x03_P4.20mm_Vertical, F.Cu at (400.9, 91.3)
- added J8: 1217080-1, SamacSys_Parts:1217080-1, F.Cu at (162.5, 90.0)
- added J8: MiniFit_2x02_F, Connector_Molex:Molex_Mini-Fit_Jr_5566-04A_2x02_P4.20mm_Vertical, F.Cu at (468.8, 69.5)
- added Q5: 2N7002, Package_TO_SOT_SMD:SOT-23, F.Cu at (399.6, 40.4)
- added Q6: BS250, Package_TO_SOT_THT:TO-92_Inline, F.Cu at (457.8, 22.7)
- added Q7: 2N7002, Package_TO_SOT_SMD:SOT-23, F.Cu at (467.7, 13.9)
- added Q8: 2N7002, Package_TO_SOT_SMD:SOT-23, F.Cu at (120.3, 138.7)
- D1, D3, D6: value BZX79C2V7 -> US1M; footprint Diode_SMD:D_MiniMELF -> Diode_SMD:D_SMA
- D10: value SS34 -> US1M; footprint Diode_SMD:D_SMC_Handsoldering -> Diode_SMD:D_SMA
- D4, D5: value SK510 -> BZX79C2V7; footprint Diode_SMD:D_SMB_Handsoldering -> Diode_SMD:D_MiniMELF
- D7: value US1M -> P600A; footprint Diode_SMD:D_SMA -> Diode_THT:D_P600_R-6_P12.70mm_Horizontal
- D8: value BZX79C2V7 -> P600A; footprint Diode_SMD:D_MiniMELF -> Diode_THT:D_P600_R-6_P12.70mm_Horizontal
- D9: value US1M -> BZX79C2V7; footprint Diode_SMD:D_SMA -> Diode_SMD:D_MiniMELF
- J1: value XT60-M -> XT60L-F; footprint Connector_AMASS:AMASS_XT60PW-M_1x02_P7.20mm_Horizontal -> Connector_AMASS:AMASS_XT60-M_1x02_P7.20mm_Vertical
- J12, J9: value 1-726388-2 -> 1217080-1; footprint SamacSys_Parts:17263882 -> SamacSys_Parts:1217080-1
- J4: value Barrel_Jack -> MiniFit_2x03_F; footprint Connector_BarrelJack:BarrelJack_CUI_PJ-063AH_Horizontal -> Connector_Molex:Molex_Mini-Fit_Jr_5566-06A_2x03_P4.20mm_Vertical
- K1, K2, K3: value RAYEX-L90S -> FINDER-40.61; footprint Relay_THT:Relay_SPDT_RAYEX-L90S -> Relay_THT:Relay_DPDT_Finder_40.52
- Q3: value 2N7002 -> BS250; footprint Package_TO_SOT_SMD:SOT-23 -> Package_TO_SOT_THT:TO-92_Inline
- R10, R11, R12, R13, R8, R9: value 10K -> 470R; footprint Resistor_SMD:R_1206_3216Metric_Pad1.30x1.75mm_HandSolder -> Resistor_THT:R_Axial_DIN0204_L3.6mm_D1.6mm_P5.08mm_Horizontal
- R14, R15: value 1.5K -> 470R; footprint Resistor_SMD:R_1206_3216Metric_Pad1.30x1.75mm_HandSolder -> Resistor_THT:R_Axial_DIN0204_L3.6mm_D1.6mm_P5.08mm_Horizontal
- R16: value 3.6K -> 10K
- R17: value 11K -> 10K; footprint Resistor_THT:R_Axial_DIN0204_L3.6mm_D1.6mm_P5.08mm_Horizontal -> Resistor_SMD:R_1206_3216Metric_Pad1.30x1.75mm_HandSolder
- R3: value 15K -> 1K
- R5, R6: value 15K -> 10K
- R7: value 15K -> 470R; footprint Resistor_SMD:R_1206_3216Metric_Pad1.30x1.75mm_HandSolder -> Resistor_THT:R_Axial_DIN0204_L3.6mm_D1.6mm_P5.08mm_Horizontal
- U1: value ATtiny84-20P -> LM555xN; footprint Package_DIP:DIP-14_W7.62mm -> Package_DIP:DIP-8_W7.62mm
- moved R11 448.5 mm to (462.3, 96.7)
- moved R14 439.5 mm to (462.3, 103.0)
- moved R15 436.9 mm to (462.3, 90.3)
- moved D8 411.2 mm to (438.7, 12.6), turned to 0 degrees
- moved D6 404.5 mm to (432.3, 12.5), turned to 0 degrees
- moved R10 398.1 mm to (414.5, 67.4)
- moved R8 397.8 mm to (414.5, 61.1), turned to 0 degrees
- moved R6 397.3 mm to (448.8, 38.7)
- moved R5 396.3 mm to (448.8, 35.4), turned to 0 degrees
- moved Q3 387.6 mm to (421.2, 28.1)
- moved Q4 365.8 mm to (399.6, 36.0)
- moved R7 362.2 mm to (414.5, 58.0)
- moved U1 350.9 mm to (410.0, 26.9), turned to 0 degrees
- moved R12 259.9 mm to (462.3, 99.8), turned to 0 degrees
- moved R16 258.4 mm to (465.3, 24.4), turned to 0 degrees
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Connections:
- D1 pad 1: Net-(D1-K) -> AuxSwitch
- D1 pad 2: GND -> Net-(D1-A)
- D10 pad 2: GND -> Net-(D10-A)
- D2 pad 1: +BATT -> AuxSwitch
- D3 pad 1: Net-(D3-K) -> AuxBeams
- D3 pad 2: GND -> AuxHBeam
- D4 pad 1: RBlinker -> Net-(D4-K)
- D4 pad 2: EBlinker -> GND
- D5 pad 1: LBlinker -> Net-(D5-K)
- D5 pad 2: EBlinker -> GND
- D6 pad 1: Net-(D6-K) -> AuxBeams
- D6 pad 2: GND -> AuxLBeam
- D7 pad 1: GND -> RBlinker
- D7 pad 2: AuxSwitch1 -> Hazard
- D8 pad 1: Net-(D8-K) -> LBlinker
- D8 pad 2: GND -> Hazard
- D9 pad 1: GND -> Net-(D9-K)
- D9 pad 2: AuxSwitch2 -> GND
- J12 pad 1: unconnected-(J12-Pad1) -> +BATT
- J12 pad 2: unconnected-(J12-Pad2) -> +BATT
- J4 pad 1: VOutlet -> VInst
- J9 pad 1: VRadio -> +12V
- J9 pad 2: VRadio -> +12V
- K1 pad 11: +12V -> AuxLBeam
- K1 pad 14: +BATT -> VLight
- K1 pad A1: +BATT -> AuxSwitch
- K1 pad A2: Net-(D2-A) -> Net-(D1-A)
- K2 pad 11: ABeam1 -> AuxHBeam
- K2 pad A1: GND -> AuxSwitch
- K2 pad A2: AuxSwitch1 -> Net-(D2-A)
- K3 pad 11: ABeam2 -> +12V
- K3 pad 14: VLight -> +BATT
- K3 pad A1: GND -> +BATT
- K3 pad A2: AuxSwitch2 -> Net-(D28-A)
- Q1 pad 1: Net-(D1-K) -> Net-(D4-K)
- Q1 pad 2: Net-(Q1-S) -> GND
- Q1 pad 3: Net-(D2-A) -> Net-(D1-A)
- Q2 pad 1: Net-(D3-K) -> Net-(D5-K)
- Q2 pad 3: Net-(Q1-S) -> Net-(D2-A)
- Q3 pad 1: Net-(D6-K) -> VInst
- Q3 pad 2: GND -> Net-(D9-K)
- Q3 pad 3: GND1 -> HazardLed
- Q4 pad 1: Net-(D8-K) -> Net-(D9-K)
- Q4 pad 3: GND2 -> HazardLed
- R1 pad 1: Net-(D1-K) -> LBeam
- R1 pad 2: Killswitch -> Net-(D4-K)
- R10 pad 1: GND -> Net-(D16-A)
- R10 pad 2: EBlinkerSensor -> VInst
- R11 pad 1: GND -> Net-(D17-A)
- R11 pad 2: EBlinkerSensor -> LBlinker
- R12 pad 1: GND -> Net-(D18-A)
- R12 pad 2: Net-(JP1-B) -> HBeam
- R13 pad 1: GND -> Net-(D19-A)
- R13 pad 2: Net-(JP1-B) -> HazardLed
- R14 pad 2: Net-(D6-K) -> AuxBeams
- R15 pad 2: Net-(D8-K) -> RBlinker
- R16 pad 1: Net-(U2-FB) -> VRadioBackup
- R16 pad 2: GND -> Net-(D26-K)
- R17 pad 1: +5V -> Key
- R17 pad 2: Net-(U2-FB) -> Net-(D30-K)
- R2 pad 1: LightSensor -> HBeam
- R2 pad 2: +5V -> Net-(D5-K)
- R3 pad 1: Net-(R3-Pad1) -> Net-(D10-A)
- R3 pad 2: VInst -> +5V
- R4 pad 1: Key -> Net-(U1-Q)
- R4 pad 2: Net-(D3-K) -> Net-(D12-K)
- R5 pad 1: BatterySensor -> Hazard
- R5 pad 2: Net-(R3-Pad1) -> Net-(D9-K)
- R6 pad 1: GND -> Net-(U1-Q)
- R6 pad 2: BatterySensor -> Net-(D12-K)
- R7 pad 1: GND -> Net-(D13-A)
- R7 pad 2: BatterySensor -> VInst
- R8 pad 1: EBlinkerSensor -> Net-(D14-A)
- R8 pad 2: EBlinker -> HazardLed
- R9 pad 1: Net-(JP1-B) -> Net-(D15-A)
- R9 pad 2: PLight -> VInst
- U1 pad 1: +5V -> GND
- U1 pad 2: LightIntensityPot -> Net-(U1-THR)
- U1 pad 3: LightSensor -> Net-(U1-Q)
- U1 pad 4: RST -> +5V
- U1 pad 5: unconnected-(U1-PB2-Pad5) -> Net-(U1-CV)
- U1 pad 6: unconnected-(U1-PA7-Pad6) -> Net-(U1-THR)
- U1 pad 7: Dimmer2 -> Net-(D10-A)
- U1 pad 8: Dimmer1 -> +5V
Routing:
- net +12V: track 0.00 -> 107.8 mm
- net Killswitch: track 0.00 -> 40.2 mm
- net ABeam1: track 21.3 -> 0.00 mm
- net (no net): track 0.00 -> 20.3 mm
- net AuxSwitch1: track 19.8 -> 0.00 mm
- net AuxSwitch2: track 19.7 -> 0.00 mm
- net Net-(D2-A): track 19.5 -> 0.00 mm
- net VLight: track 42.6 -> 27.1 mm
- net ABeam2: track 8.44 -> 0.00 mm
- net AuxLBeam: track 0.00 -> 7.50 mm
- net AuxHBeam: track 0.00 -> 7.50 mm
- net +VDC: track 17.5 -> 24.2 mm
- net VRadioBackup: track 0.00 -> 5.08 mm
- net VOutlet: track 0.00 -> 5.08 mm
- net VInst: track 0.00 -> 5.08 mm
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Other:
- board text added: "5V"
- board text added: "Inst"
- board text added: "KillSwitch"
- board text added: "Lights"
- board text added: "Main"
- board text added: "Outlet"
- board text added: "Radio"
- board text added: "Spares"

Commit message: Update Schmatics; Cleanup unecessary circuits; Simplify blinkers dimmers; Update PCB; Colorize motorcycle electric diagram.
Parts:
- removed BT1: 9V, Connector_JST:JST_XH_B2B-XH-A_1x02_P2.50mm_Vertical
- removed D15, D16: LED, LED_THT:LED_D5.0mm
- removed D17, D21: LED Green, LED_THT:LED_D5.0mm
- removed D18: LED Blue, LED_THT:LED_D5.0mm
- removed D19: LED Red, LED_THT:LED_D5.0mm
- removed D20: LED Yellow, LED_THT:LED_D5.0mm
- removed D27: P600A, Diode_THT:D_P600_R-6_P12.70mm_Horizontal
- removed D28: US1M, Diode_SMD:D_SMA
- removed D30: BZX79C2V7, Diode_SMD:D_MiniMELF
- removed J** (x7), J57, J58, J59, J60, J61, J62, J63, J64, J65, J66, J67, J68: 1217080-1, SamacSys_Parts:1217080-1
- removed the J10 at (448.7, 52.1)
- removed the J10 at (142.5, 90.0)
- removed the J11 at (470.6, 52.2)
- removed the J11 at (172.5, 90.0)
- removed the J13 at (132.5, 101.8)
- removed the J13 at (448.7, 65.2)
- removed the J14 at (448.7, 105.1)
- removed the J14 at (162.5, 101.8)
- removed the J15 at (152.5, 101.7)
- removed the J15 at (456.2, 105.1)
- removed the J16 at (448.7, 92.0)
- removed the J16 at (142.5, 101.6)
- removed the J4 at (400.9, 52.1)
- removed J42, J48: MiniFit_2x04_M, Connector_Molex:Molex_Mini-Fit_Jr_5566-08A_2x04_P4.20mm_Vertical
- removed J44: MiniFit_2x02_M, Connector_Molex:Molex_Mini-Fit_Jr_5566-04A_2x02_P4.20mm_Vertical
- removed J45, J46, J47, J49, J50: MiniFit_2x03_M, Connector_Molex:Molex_Mini-Fit_Jr_5566-06A_2x03_P4.20mm_Vertical
- removed J51, J55: MiniFit_2x01_F, Connector_Molex:Molex_Mini-Fit_Jr_5566-02A_2x01_P4.20mm_Vertical
- removed J53, J54: Barrel_Jack, Connector_BarrelJack:BarrelJack_CUI_PJ-063AH_Horizontal
- removed the J6 at (400.9, 78.2)
- removed the J6 at (122.5, 101.7)
- removed the J7 at (132.5, 90.0)
- removed the J7 at (400.9, 91.3)
- removed the J8 at (162.5, 90.0)
- removed the J8 at (468.8, 69.5)
- removed Q8: 2N7002, Package_TO_SOT_SMD:SOT-23
- removed R10, R11, R12, R13, R14, R15, R9: 470R, Resistor_THT:R_Axial_DIN0204_L3.6mm_D1.6mm_P5.08mm_Horizontal
- removed R16, R17: 10K, Resistor_SMD:R_1206_3216Metric_Pad1.30x1.75mm_HandSolder
- added D24: US1M, Diode_SMD:D_SMA, B.Cu at (130.7, 100.0)
- added D25: 2.7V, Diode_SMD:D_MiniMELF, B.Cu at (130.7, 103.5)
- added IC1: SN74LVC1G86DBVT, SamacSys_Parts:SOT95P280X145-5N, F.Cu at (181.3, 136.6)
- added J10: Conn_01x01_Socket, Connector_Pin:Pin_D1.0mm_L10.0mm, B.Cu at (138.0, 77.2)
- added J11: Conn_01x01_Socket, Connector_Pin:Pin_D1.0mm_L10.0mm, B.Cu at (142.2, 77.2)
- added J13: Conn_01x01_Socket, Connector_Pin:Pin_D1.0mm_L10.0mm, B.Cu at (108.5, 61.8)
- added J14: Conn_01x01_Socket, Connector_Pin:Pin_D1.0mm_L10.0mm, B.Cu at (112.7, 61.8)
- added J15: Conn_01x01_Socket, Connector_Pin:Pin_D1.0mm_L10.0mm, B.Cu at (117.0, 61.8)
- added J16: Conn_01x01_Socket, Connector_Pin:Pin_D1.0mm_L10.0mm, B.Cu at (121.2, 61.8)
- added J18: Conn_01x01_Socket, Connector_Pin:Pin_D1.0mm_L10.0mm, B.Cu at (129.6, 61.8)
- added J19: Conn_01x01_Socket, Connector_Pin:Pin_D1.0mm_L10.0mm, B.Cu at (133.8, 61.8)
- added J20: Conn_01x01_Socket, Connector_Pin:Pin_D1.0mm_L10.0mm, B.Cu at (138.1, 61.8)
- added J21: Conn_01x01_Socket, Connector_Pin:Pin_D1.0mm_L10.0mm, B.Cu at (142.3, 61.8)
- added J22: Conn_01x01_Socket, Connector_Pin:Pin_D1.0mm_L10.0mm, B.Cu at (146.5, 61.8)
- added J23: Conn_01x01_Socket, Connector_Pin:Pin_D1.0mm_L10.0mm, F.Cu at (172.4, 86.7)
- added J24: Conn_01x01_Socket, Connector_Pin:Pin_D1.0mm_L10.0mm, F.Cu at (167.2, 113.4)
- added J25: Conn_01x01_Socket, Connector_Pin:Pin_D1.0mm_L10.0mm, F.Cu at (154.4, 86.7)
- added J26: Conn_01x01_Socket, Connector_Pin:Pin_D1.0mm_L10.0mm, F.Cu at (149.2, 113.4)
- added J27: Conn_01x01_Socket, Connector_Pin:Pin_D1.0mm_L10.0mm, F.Cu at (163.4, 86.4)
- added J28: Conn_01x01_Socket, Connector_Pin:Pin_D1.0mm_L10.0mm, F.Cu at (159.9, 113.4)
- added J29: Conn_01x01_Socket, Connector_Pin:Pin_D1.0mm_L10.0mm, F.Cu at (150.9, 145.8)
- added J3: Conn_01x01_Socket, Connector_Pin:Pin_D1.0mm_L10.0mm, B.Cu at (108.6, 77.2)
- added J30: Conn_01x01_Socket, Connector_Pin:Pin_D1.0mm_L10.0mm, F.Cu at (150.9, 149.9)
- added J31: Conn_01x01_Socket, Connector_Pin:Pin_D1.0mm_L10.0mm, F.Cu at (155.0, 145.8)
- added J32: Conn_01x01_Socket, Connector_Pin:Pin_D1.0mm_L10.0mm, F.Cu at (155.0, 149.9)
- added J33: Conn_01x01_Socket, Connector_Pin:Pin_D1.0mm_L10.0mm, F.Cu at (123.5, 113.5)
- added J34: Conn_01x01_Socket, Connector_Pin:Pin_D1.0mm_L10.0mm, F.Cu at (159.1, 145.8)
- added J35: Conn_01x01_Socket, Connector_Pin:Pin_D1.0mm_L10.0mm, F.Cu at (154.7, 113.4)
- added J36: Conn_01x01_Socket, Connector_Pin:Pin_D1.0mm_L10.0mm, F.Cu at (159.1, 149.9)
- added J37: Conn_01x01_Socket, Connector_Pin:Pin_D1.0mm_L10.0mm, F.Cu at (129.2, 113.5)
- added J38: Conn_01x01_Socket, Connector_Pin:Pin_D1.0mm_L10.0mm, F.Cu at (163.1, 145.8)
- added J39: Conn_01x01_Socket, Connector_Pin:Pin_D1.0mm_L10.0mm, F.Cu at (163.1, 149.9)
- added J4: 1217080-1, SamacSys_Parts:1217080-1, F.Cu at (125.0, 150.8)
- added J4: Conn_01x01_Socket, Connector_Pin:Pin_D1.0mm_L10.0mm, B.Cu at (112.8, 77.2)
- added J40: Conn_01x01_Socket, Connector_Pin:Pin_D1.0mm_L10.0mm, F.Cu at (108.0, 106.0)
- added J6: Conn_01x01_Socket, Connector_Pin:Pin_D1.0mm_L10.0mm, B.Cu at (121.2, 77.2)
- added J7: Conn_01x01_Socket, Connector_Pin:Pin_D1.0mm_L10.0mm, B.Cu at (125.4, 77.2)
- added J8: Conn_01x01_Socket, Connector_Pin:Pin_D1.0mm_L10.0mm, B.Cu at (129.6, 77.2)
- added J96: Conn_01x01_Socket, Connector_Pin:Pin_D1.0mm_L10.0mm, F.Cu at (118.2, 142.2)
- added J97: Conn_01x01_Socket, Connector_Pin:Pin_D1.0mm_L10.0mm, F.Cu at (111.0, 142.0)
- added R18: 10K, Resistor_SMD:R_1206_3216Metric_Pad1.30x1.75mm_HandSolder, B.Cu at (125.0, 103.5)
- added R19: 100, Resistor_SMD:R_1206_3216Metric_Pad1.30x1.75mm_HandSolder, F.Cu at (108.8, 100.5)
- added R20: 1.5K, Resistor_SMD:R_1206_3216Metric_Pad1.30x1.75mm_HandSolder, F.Cu at (103.3, 95.3)
- added R21: 10K, Resistor_SMD:R_1206_3216Metric_Pad1.30x1.75mm_HandSolder, F.Cu at (103.5, 100.8)
- D10, Q4, R5: moved to B.Cu
- D11, D3: value US1M -> 2.7V; footprint Diode_SMD:D_SMA -> Diode_SMD:D_MiniMELF
- D12, D5, D9: value BZX79C2V7 -> US1M; footprint Diode_SMD:D_MiniMELF -> Diode_SMD:D_SMA; moved to B.Cu
- D13: value LED -> 2.7V; footprint LED_THT:LED_D5.0mm -> Diode_SMD:D_MiniMELF; moved to B.Cu
- D14: value LED -> 2.7V; footprint LED_THT:LED_D5.0mm -> Diode_SMD:D_MiniMELF
- D26: value BZX79C2V7 -> 10V
- D4: value BZX79C2V7 -> 2.7V
- D6: value US1M -> 2.7V; footprint Diode_SMD:D_SMA -> Diode_SMD:D_MiniMELF; moved to B.Cu
- J1: renamed from J2; footprint Connector_AMASS:AMASS_XT60PW-M_1x02_P7.20mm_Horizontal -> Local Footprints:AMASS_XT60PW-M_1x02_P7.20mm_Horizontal_Short
- J1: value XT60L-F -> MiniFit_2x10_F; footprint Connector_AMASS:AMASS_XT60-M_1x02_P7.20mm_Vertical -> Connector_Molex:Molex_Mini-Fit_Jr_5566-20A_2x10_P4.20mm_Vertical
- J12, J17, J9: value 1217080-1 -> Conn_01x01_Socket; footprint SamacSys_Parts:1217080-1 -> Connector_Pin:Pin_D1.0mm_L10.0mm; moved to B.Cu
- J5: value MiniFit_2x03_F -> Conn_01x01_Socket; footprint Connector_Molex:Molex_Mini-Fit_Jr_5566-06A_2x03_P4.20mm_Vertical -> Connector_Pin:Pin_D1.0mm_L10.0mm; moved to B.Cu
- K1, K2: value FINDER-40.61 -> LEG-12; footprint Relay_THT:Relay_DPDT_Finder_40.52 -> Local Footprints:LEG12
- K3: value FINDER-40.61 -> RAYEX-L90; footprint Relay_THT:Relay_DPDT_Finder_40.52 -> Local Footprints:Relay_SPDT_RAYEX-L90
- Q3, Q6: value BS250 -> 2N7002; footprint Package_TO_SOT_THT:TO-92_Inline -> Package_TO_SOT_SMD:SOT-23; moved to B.Cu
- Q7: value 2N7002 -> BC557; footprint Package_TO_SOT_SMD:SOT-23 -> Package_TO_SOT_THT:TO-92_Inline
- R1: value 10K -> 1K
- R3: value 1K -> 10K
- R7: value 470R -> 10K; footprint Resistor_THT:R_Axial_DIN0204_L3.6mm_D1.6mm_P5.08mm_Horizontal -> Resistor_SMD:R_1206_3216Metric_Pad1.30x1.75mm_HandSolder; moved to B.Cu
- R8: value 470R -> 10K; footprint Resistor_THT:R_Axial_DIN0204_L3.6mm_D1.6mm_P5.08mm_Horizontal -> Resistor_SMD:R_1206_3216Metric_Pad1.30x1.75mm_HandSolder
- moved Q7 375.4 mm to (103.2, 103.8), turned to -90 degrees
- moved D26 369.9 mm to (103.8, 98.1), turned to 180 degrees
- moved Q6 341.4 mm to (125.2, 100.0)
- moved D7 313.8 mm to (151.3, 127.8)
- moved D8 313.8 mm to (151.3, 138.5)
- moved J1 306.0 mm to (108.6, 66.6)
- moved R3 294.5 mm to (175.7, 142.5)
- moved R6 294.5 mm to (175.7, 149.1)
- moved D3 292.2 mm to (169.6, 135.9)
- moved R4 292.1 mm to (175.7, 145.8)
- moved D11 289.3 mm to (169.6, 142.6)
- moved R5 285.7 mm to (171.1, 102.4)
- moved J5 284.1 mm to (117.0, 77.2)
- moved D6 277.3 mm to (170.9, 104.9), turned to 180 degrees
- moved D10 271.4 mm to (172.7, 95.9)
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Connections:
- D1 pad 1: AuxSwitch -> Net-(D1-K)
- D10 pad 1: Net-(D10-K) -> AuxBeams
- D10 pad 2: Net-(D10-A) -> AuxLBeam
- D11 pad 1: Net-(D10-A) -> Net-(D11-K)
- D11 pad 2: Net-(D11-A) -> GND
- D12 pad 1: Net-(D12-K) -> AuxSwitch
- D12 pad 2: GND -> Net-(D12-A)
- D13 pad 1: GNDDash -> Net-(D13-K)
- D13 pad 2: Net-(D13-A) -> GND
- D14 pad 1: GNDDash -> Net-(D14-K)
- D14 pad 2: Net-(D14-A) -> GND
- D2 pad 1: AuxSwitch -> Net-(D1-A)
- D26 pad 2: GND -> Net-(D26-A)
- D3 pad 1: AuxBeams -> Net-(D3-K)
- D3 pad 2: AuxHBeam -> GND
- D4 pad 1: Net-(D4-K) -> PLightSignal
- D5 pad 1: Net-(D5-K) -> AuxSwitch
- D5 pad 2: GND -> Net-(D5-A)
- D6 pad 1: AuxBeams -> Net-(D6-K)
- D6 pad 2: AuxLBeam -> GND
- D9 pad 1: Net-(D9-K) -> AuxBeams
- D9 pad 2: GND -> AuxHBeam
- J1 pad 1: GND -> Key
- J1 pad 2: +VDC -> VRadio
- J12 pad 1: +BATT -> RBlinker
- J17 pad 1: +5V -> VLight
- J5 pad 1: HazardLed -> AuxHBeam
- J9 pad 1: +12V -> HazardLed
- K1 pad A1: AuxSwitch -> Net-(D5-A)
- K1 pad A2: Net-(D1-A) -> AuxSwitch
- K2 pad A1: AuxSwitch -> Net-(D12-A)
- K2 pad A2: Net-(D2-A) -> AuxSwitch
- K3 pad A2: Net-(D28-A) -> Net-(D24-A)
- Q1 pad 1: Net-(D4-K) -> Net-(D3-K)
- Q1 pad 3: Net-(D1-A) -> GndDimmer
- Q2 pad 1: Net-(D5-K) -> PLightSignal
- Q2 pad 2: GND -> GndDimmer
- Q2 pad 3: Net-(D2-A) -> GNDDash
- Q3 pad 1: VInst -> Net-(D6-K)
- Q3 pad 2: Net-(D9-K) -> GND
- Q3 pad 3: HazardLed -> Net-(D5-A)
- Q4 pad 1: Net-(D9-K) -> Net-(D13-K)
- Q4 pad 3: HazardLed -> Net-(D12-A)
- Q5 pad 1: Net-(D12-K) -> Net-(D14-K)
- Q5 pad 2: GND -> HazardLed
- Q5 pad 3: GNDDash -> GndDimmer
- Q6 pad 2: Net-(D26-K) -> GND
- Q6 pad 3: Net-(D25-A) -> Net-(D24-A)
- Q7 pad 1: Net-(D26-K) -> +BATT
- Q7 pad 2: GND -> Net-(D26-A)
- Q7 pad 3: Net-(D25-A) -> LowBat
- R1 pad 1: LBeam -> Net-(D1-A)
- R1 pad 2: Net-(D4-K) -> +5V
- R2 pad 1: HBeam -> Net-(U1-Q)
- R2 pad 2: Net-(D5-K) -> Net-(D3-K)
- R3 pad 1: Net-(D10-A) -> Net-(U1-Q)
- R3 pad 2: +5V -> Net-(D3-K)
- R4 pad 1: Net-(U1-Q) -> PLight
- R4 pad 2: Net-(D12-K) -> PLightSignal
- R5 pad 1: Hazard -> LBeam
- R5 pad 2: Net-(D9-K) -> Net-(D6-K)
- R6 pad 1: Net-(U1-Q) -> Hazard
- R6 pad 2: Net-(D12-K) -> Net-(D11-K)
- R7 pad 1: Net-(D13-A) -> HBeam
- R7 pad 2: VInst -> Net-(D13-K)
- R8 pad 1: Net-(D14-A) -> Net-(IC1-Y)
- R8 pad 2: HazardLed -> Net-(D14-K)
- U1 pad 7: Net-(D10-A) -> Net-(D1-A)
Routing:
- net +12V: track 107.8 -> 18.9 mm
- net AuxSwitch: track 0.00 -> 58.0 mm
- net Killswitch: track 40.2 -> 0.00 mm
- net AuxBeams: track 0.00 -> 24.8 mm
- net (no net): track 20.3 -> 0.00 mm, vias 0 -> 5
- net +VDC: track 24.2 -> 6.00 mm, vias 0 -> 1
- net Net-(D24-A): track 0.00 -> 18.0 mm
- net +BATT: track 69.9 -> 52.0 mm
- net HBeam: track 0.00 -> 17.4 mm
- net LBeam: track 0.00 -> 15.8 mm
- net Net-(D12-A): track 0.00 -> 10.4 mm
- net Net-(D5-A): track 0.00 -> 10.3 mm
- net Key: track 0.00 -> 10.0 mm
- net Net-(D26-A): track 0.00 -> 8.07 mm
- net Net-(D13-K): track 0.00 -> 7.50 mm
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- removed copper zone on F.Cu, net GND
Other:
- board outline added: 100 x 97 mm
- board text removed: "5V"
- board text removed: "Inst"
- board text removed: "KillSwitch"
- board text removed: "Lights"
- board text removed: "Main"
- board text removed: "Outlet"
- board text removed: "Radio"
- board text removed: "Spares"

Commit message: Update Schematics; Replace xor with quad nand; Update PCB
Parts:
- removed IC1: SN74LVC1G86DBVT, SamacSys_Parts:SOT95P280X145-5N
- added D10: US1M, Diode_SMD:D_SMA, F.Cu at (106.8, 108.5)
- added D17: LED, LED_THT:LED_D5.0mm, F.Cu at (431.9, -75.3)
- added D18: LED, LED_THT:LED_D5.0mm, F.Cu at (439.4, -75.3)
- added D19: LED, LED_THT:LED_D5.0mm, F.Cu at (446.9, -75.3)
- added D20: LED, LED_THT:LED_D5.0mm, F.Cu at (454.4, -75.3)
- added D21: LED Green, LED_THT:LED_D5.0mm, F.Cu at (372.1, -8.07)
- added D22: LED Blue, LED_THT:LED_D5.0mm, F.Cu at (379.6, -8.07)
- added D23: LED Red, LED_THT:LED_D5.0mm, F.Cu at (387.1, -8.07)
- added D24: LED Yellow, LED_THT:LED_D5.0mm, F.Cu at (394.6, -8.07)
- added D25: LED Green, LED_THT:LED_D5.0mm, F.Cu at (402.1, -8.07)
- added D9: US1M, Diode_SMD:D_SMA, F.Cu at (106.8, 103.5)
- added J100: Conn_01x01_Socket, Connector_Pin:Pin_D1.0mm_L10.0mm, F.Cu at (136.5, 86.8)
- added J101: 1217080-1, SamacSys_Parts:1217080-1, F.Cu at (465.7, -77.5)
- added J102: 1217080-1, SamacSys_Parts:1217080-1, F.Cu at (465.7, -74.3)
- added J103: 1217080-1, SamacSys_Parts:1217080-1, F.Cu at (465.7, -71.1)
- added J104: 1217080-1, SamacSys_Parts:1217080-1, F.Cu at (465.7, -67.9)
- added J105: 1217080-1, SamacSys_Parts:1217080-1, F.Cu at (465.7, -64.7)
- added J106: 1217080-1, SamacSys_Parts:1217080-1, F.Cu at (465.7, -61.5)
- added J107: 1217080-1, SamacSys_Parts:1217080-1, F.Cu at (465.7, -58.3)
- added J108: 1217080-1, SamacSys_Parts:1217080-1, F.Cu at (465.7, -55.1)
- added J109: 1217080-1, SamacSys_Parts:1217080-1, F.Cu at (465.7, -51.9)
- added J110: 1217080-1, SamacSys_Parts:1217080-1, F.Cu at (465.7, -48.7)
- added J111: 1217080-1, SamacSys_Parts:1217080-1, F.Cu at (465.7, -45.5)
- added J112: 1217080-1, SamacSys_Parts:1217080-1, F.Cu at (465.7, -42.3)
- added J41: MiniFit_2x03_F, Connector_Molex:Molex_Mini-Fit_Jr_5566-06A_2x03_P4.20mm_Vertical, F.Cu at (417.3, -75.8)
- added J42: MiniFit_2x03_F, Connector_Molex:Molex_Mini-Fit_Jr_5566-06A_2x03_P4.20mm_Vertical, F.Cu at (417.3, -62.8)
- added J43: MiniFit_2x03_F, Connector_Molex:Molex_Mini-Fit_Jr_5566-06A_2x03_P4.20mm_Vertical, F.Cu at (417.3, -49.7)
- added J44: MiniFit_2x03_F, Connector_Molex:Molex_Mini-Fit_Jr_5566-06A_2x03_P4.20mm_Vertical, F.Cu at (417.3, -36.7)
- added J45: MiniFit_2x04_M, Connector_Molex:Molex_Mini-Fit_Jr_5566-08A_2x04_P4.20mm_Vertical, F.Cu at (417.3, -21.6)
- added J46: MiniFit_2x02_F, Connector_Molex:Molex_Mini-Fit_Jr_5566-04A_2x02_P4.20mm_Vertical, F.Cu at (437.3, -4.32)
- added J47: MiniFit_2x04_F, Connector_Molex:Molex_Mini-Fit_Jr_5566-08A_2x04_P4.20mm_Vertical, F.Cu at (417.3, -8.57)
- added J50: USB_A, Connector_USB:USB_A_Molex_67643_Horizontal, F.Cu at (439.2, -21.6)
- added J51: MiniFit_2x01_M, Connector_Molex:Molex_Mini-Fit_Jr_5566-02A_2x01_P4.20mm_Vertical, F.Cu at (373.3, 12.0)
- added J52: MiniFit_2x01_M, Connector_Molex:Molex_Mini-Fit_Jr_5566-02A_2x01_P4.20mm_Vertical, F.Cu at (380.8, 12.0)
- added J53: MiniFit_2x03_F, Connector_Molex:Molex_Mini-Fit_Jr_5566-06A_2x03_P4.20mm_Vertical, F.Cu at (373.3, -1.02)
- added J69: MiniFit_2x04_M, Connector_Molex:Molex_Mini-Fit_Jr_5566-08A_2x04_P4.20mm_Vertical, F.Cu at (417.3, 10.7)
- added J84: MiniFit_2x02_M, Connector_Molex:Molex_Mini-Fit_Jr_5566-04A_2x02_P4.20mm_Vertical, F.Cu at (389.2, -34.7)
- added J85: MiniFit_2x03_M, Connector_Molex:Molex_Mini-Fit_Jr_5566-06A_2x03_P4.20mm_Vertical, F.Cu at (373.3, -75.8)
- added J86: MiniFit_2x01_F, Connector_Molex:Molex_Mini-Fit_Jr_5566-02A_2x01_P4.20mm_Vertical, F.Cu at (389.2, -47.7)
- added J87: MiniFit_2x01_F, Connector_Molex:Molex_Mini-Fit_Jr_5566-02A_2x01_P4.20mm_Vertical, F.Cu at (396.6, -47.7)
- added J88: MiniFit_2x04_M, Connector_Molex:Molex_Mini-Fit_Jr_5566-08A_2x04_P4.20mm_Vertical, F.Cu at (389.2, -60.8)
- added J89: 1217080-1, SamacSys_Parts:1217080-1, F.Cu at (389.8, -23.3)
- added J91: Barrel_Jack, Connector_BarrelJack:BarrelJack_CUI_PJ-063AH_Horizontal, F.Cu at (392.0, -77.1)
- added J92: MiniFit_2x03_M, Connector_Molex:Molex_Mini-Fit_Jr_5566-06A_2x03_P4.20mm_Vertical, F.Cu at (373.3, -62.8)
- added J93: MiniFit_2x03_M, Connector_Molex:Molex_Mini-Fit_Jr_5566-06A_2x03_P4.20mm_Vertical, F.Cu at (373.3, -49.7)
- added J94: Barrel_Jack, Connector_BarrelJack:BarrelJack_CUI_PJ-063AH_Horizontal, F.Cu at (405.0, -77.1)
- added J96: MiniFit_2x03_M, Connector_Molex:Molex_Mini-Fit_Jr_5566-06A_2x03_P4.20mm_Vertical, F.Cu at (373.3, -36.7)
- added J97: MiniFit_2x03_M, Connector_Molex:Molex_Mini-Fit_Jr_5566-06A_2x03_P4.20mm_Vertical, F.Cu at (373.3, -23.6)
- added R10: 470R, Resistor_THT:R_Axial_DIN0204_L3.6mm_D1.6mm_P5.08mm_Horizontal, F.Cu at (430.9, -63.7)
- added R11: 470R, Resistor_THT:R_Axial_DIN0204_L3.6mm_D1.6mm_P5.08mm_Horizontal, F.Cu at (430.9, -60.5)
- added R12: 680R, Resistor_THT:R_Axial_DIN0204_L3.6mm_D1.6mm_P5.08mm_Horizontal, F.Cu at (386.9, -2.73)
- added R13: 680R, Resistor_THT:R_Axial_DIN0204_L3.6mm_D1.6mm_P5.08mm_Horizontal, F.Cu at (386.9, 0.42)
- added R14: 680R, Resistor_THT:R_Axial_DIN0204_L3.6mm_D1.6mm_P5.08mm_Horizontal, F.Cu at (386.9, 3.58)
- added R15: 680R, Resistor_THT:R_Axial_DIN0204_L3.6mm_D1.6mm_P5.08mm_Horizontal, F.Cu at (386.9, 6.72)
- added R16: 680R, Resistor_THT:R_Axial_DIN0204_L3.6mm_D1.6mm_P5.08mm_Horizontal, F.Cu at (386.9, 9.88)
- added R2: 1K, Resistor_SMD:R_1206_3216Metric_Pad1.30x1.75mm_HandSolder, B.Cu at (132.6, 117.8)
- added R8: 470R, Resistor_THT:R_Axial_DIN0204_L3.6mm_D1.6mm_P5.08mm_Horizontal, F.Cu at (430.9, -70.0)
- added R9: 470R, Resistor_THT:R_Axial_DIN0204_L3.6mm_D1.6mm_P5.08mm_Horizontal, F.Cu at (430.9, -66.8)
- added U2: 74LS00, Package_DIP:DIP-14_W7.62mm_Socket_LongPads, F.Cu at (114.2, 113.5)
- D16: renamed from D14; moved to B.Cu
- D3, Q1, Q2, Q5, R1, R2, R3: moved to B.Cu
- D7, D8: value P600A -> US1M; footprint Diode_THT:D_P600_R-6_P12.70mm_Horizontal -> Diode_SMD:D_SMA
- R7: renamed from R8; moved to B.Cu
- U1: footprint Package_DIP:DIP-8_W7.62mm -> Package_DIP:DIP-8_W7.62mm_Socket_LongPads
- moved Q5 79.1 mm to (107.1, 122.2), turned to 180 degrees
- moved R5 77.5 mm to (108.0, 111.5)
- moved J32 76.3 mm to (101.0, 96.0)
- moved J30 69.8 mm to (101.0, 101.1)
- moved R7 69.7 mm to (111.4, 125.5), turned to 90 degrees
- moved D13 68.1 mm to (107.8, 114.0), turned to 180 degrees
- moved J31 67.1 mm to (101.0, 106.0)
- moved D16 63.7 mm to (111.4, 120.0), turned to 90 degrees
- moved J34 61.0 mm to (186.2, 91.2), turned to 90 degrees
- moved D8 59.9 mm to (106.8, 98.5)
- moved Q2 59.2 mm to (127.3, 121.0), turned to 180 degrees
- moved Q1 56.4 mm to (127.3, 124.5), turned to 180 degrees
- moved R3 56.4 mm to (126.3, 118.8), turned to 180 degrees
- moved D7 56.3 mm to (106.8, 93.3)
- moved J39 50.6 mm to (128.8, 112.8)
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- renumbered D9 to D11, D10 to D12, D11 to D13, D12 to D14, D13 to D15, D24 to D26, D25 to D27, D26 to D28, J96 to J98, J97 to J99, R18 to R17, R19 to R18, R20 to R19, R21 to R20, R4 to R3, R5 to R4, R6 to R5, R7 to R6
Connections:
- net Net-(D11-K) renamed /Main board/XOR 74LS00/B
- D8 pad 1: LBlinker -> RBlinker
- K1 pad NC: unconnected-(K1-PadNC) -> GND
- K2 pad NC: unconnected-(K2-PadNC) -> GND
- R7 pad 1: Net-(IC1-Y) -> /Main board/XOR 74LS00/O
Routing:
- net GndDimmer: track 0.00 -> 46.7 mm
- net LBeam: track 15.8 -> 53.0 mm
- net Key: track 10.0 -> 38.4 mm
- net Hazard: track 0.00 -> 26.5 mm
- net Net-(U2-Pad13): track 0.00 -> 19.4 mm
- net /Main board/XOR 74LS00/B: track 0.00 -> 18.9 mm
- net +5V: track 0.00 -> 17.6 mm
- net PLightSignal: track 0.00 -> 14.4 mm
- net +BATT: track 52.0 -> 66.2 mm
- net Net-(D3-K): track 0.00 -> 13.8 mm
- net VLight: track 29.4 -> 43.0 mm
- net Net-(D1-A): track 0.00 -> 11.0 mm
- net Net-(U2-Pad5): track 0.00 -> 9.72 mm
- net Net-(U1-THR): track 0.00 -> 8.67 mm
- net LowBat: track 4.85 -> 13.3 mm
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