File: src/dragstar-infotainment.kicad_pcb (KiCad board)
At the start: 2 copper layers, 75 x 100 mm, 76 parts, among them J10 Conn_01x01, J11 Conn_01x01, J12 Conn_01x01, J13 Conn_01x01, J14 Conn_01x01, J15 Conn_01x01, J16 Conn_01x01, J17 Conn_01x01, J18 Conn_01x01, J19 Conn_01x01, J20 Conn_01x01, J21 Conn_01x01, J22 Conn_01x01, J23 XT60-M, J24 Conn_01x01, J25 Conn_01x01, J26 1217080-1, J27 1217080-1, J28 1217080-1, J29 1217080-1, J3 Conn_01x01, J30 1217080-1, J31 1217080-1, J32 1217080-1, J33 1217080-1, J34 1217080-1, J35 1217080-1, J4 Conn_01x01, J5 Conn_01x01, J6 Conn_01x01, J7 Conn_01x01, J8 Conn_01x01, J9 Conn_01x01, K1 RAYEX-L90, K2 LEG-12, K3 LEG-12, Q1 2N7002, Q2 2N7002, Q3 2N7002, Q4 2N7002, Q5 2N7002, Q6 2N7002

Commit message: PCB Layout adjustments; generate new plots
Parts:
- moved R6 23.4 mm to (144.0, 142.8), turned to -90 degrees
- moved RV1 16.6 mm to (147.0, 142.8), turned to 0 degrees
- moved J16 16.2 mm to (142.0, 132.5)
- moved R5 13.5 mm to (157.5, 133.8), turned to -90 degrees
- moved R3 13.2 mm to (146.9, 138.8), turned to 0 degrees
- moved J3 13.0 mm to (127.0, 144.5)
- moved R4 12.6 mm to (150.9, 132.2), turned to 0 degrees
- moved Q4 12.3 mm to (150.0, 141.2)
- moved D12 11.0 mm to (155.0, 138.5), turned to 90 degrees
- moved Q3 10.2 mm to (148.6, 135.3), turned to 90 degrees
- moved J19 9.13 mm to (140.5, 144.5)
- moved D3 6.56 mm to (133.8, 144.5)
- moved Q2 6.56 mm to (136.5, 140.8)
- moved R2 6.56 mm to (131.4, 140.3)
- moved R17 6.43 mm to (152.0, 137.2), turned to 90 degrees
Routing:
- net VInst: track 36.1 -> 29.0 mm
- net PLight: track 13.0 -> 17.8 mm
- net Net-(D12-A): track 7.24 -> 10.8 mm
- net Net-(Q3-G): track 10.8 -> 7.56 mm
- net RBlinker: track 67.8 -> 71.1 mm
- net Net-(D12-K): track 9.20 -> 5.95 mm
- net Net-(R4-Pad1): track 5.36 -> 2.61 mm
- net LowBat: track 6.15 -> 7.65 mm
- net Net-(R6-Pad2): track 2.50 -> 3.64 mm
- net LBlinker: track 65.6 -> 66.3 mm
